Commit message: change objects urdf and paths

File: assets/objects/sphere3.urdf (robot description, URDF)
Before this commit: robot urdf_robot, 1 links, 0 joints
Links:
- link base_link: geometry collision sphere radius=0.003; visual mesh filename=textured_sphere_smooth.obj scale=0.003 0.003 0.003

File: assets/objects/sphere4.urdf (robot description, URDF)
Before this commit: robot urdf_robot, 1 links, 0 joints
Links:
- link base_link: geometry collision sphere radius=0.004; visual mesh filename=textured_sphere_smooth.obj scale=0.004 0.004 0.004

File: assets/objects/sphere5.urdf (robot description, URDF)
Before this commit: robot urdf_robot, 1 links, 0 joints
Links:
- link base_link: geometry collision sphere radius=0.005; visual mesh filename=textured_sphere_smooth.obj scale=0.005 0.005 0.005

Commit message: fix urdf objects

File: assets/objects/sphere3.urdf (robot description, URDF)
Before this commit: robot urdf_robot, 1 links, 0 joints
Links:
- link base_link: geometry collision sphere radius=0.015; visual mesh filename=textured_sphere_smooth.obj scale=0.015 0.015 0.015

File: assets/objects/sphere4.urdf (robot description, URDF)
Before this commit: robot urdf_robot, 1 links, 0 joints
Links:
- link base_link: geometry collision sphere radius=0.02; visual mesh filename=textured_sphere_smooth.obj scale=0.02 0.02 0.02

File: assets/objects/sphere5.urdf (robot description, URDF)
Before this commit: robot urdf_robot, 1 links, 0 joints
Links:
- link base_link: geometry collision sphere radius=0.025; visual mesh filename=textured_sphere_smooth.obj scale=0.025 0.025 0.025

Commit message: fix collect issues

File: assets/objects/sphere3.urdf (robot description, URDF)
Before this commit: robot urdf_robot, 1 links, 0 joints
Links:
- link base_link: geometry collision sphere radius=0.003; visual mesh filename=textured_sphere_smooth.obj scale=0.003 0.003 0.003
