Commit message: oshers games

File: assets/objects/rect_small.urdf (robot description, URDF)
Before this commit: robot cube.urdf, 1 links, 0 joints
Links:
- link baseLink: mass 1 -> 0.01; geometry collision box size=.04 .02 .07; visual mesh filename=cube.obj scale=.04 .02 .07

File: assets/objects/sphere_small.urdf (robot description, URDF)
Before this commit: robot urdf_robot, 1 links, 0 joints
Links:
- link base_link: mass .1 -> 0.1; geometry collision sphere radius=0.04; visual mesh filename=textured_sphere_smooth.obj scale=0.04 0.04 0.04
