Commit message: update obj files

File: assets/objects/ellipse.urdf (robot description, URDF)
Before this commit: robot urdf_robot, 1 links, 0 joints
Links:
- link base_link: geometry collision mesh filename=ellipse.obj scale=1 1 1; visual mesh filename=ellipse.obj scale=1 1 1

File: assets/objects/hexagon.urdf (robot description, URDF)
Before this commit: robot cube.urdf, 1 links, 0 joints
Links:
- link baseLink: geometry collision mesh filename=hexagon.obj scale=1 1 1; visual mesh filename=hexagon.obj scale=1 1 1

File: assets/objects/sphere3.urdf (robot description, URDF)
Before this commit: robot urdf_robot, 1 links, 0 joints
Links:
- link base_link: geometry collision mesh filename=sphere3.obj scale=1 1 1; visual mesh filename=sphere3.obj scale=1 1 1

File: assets/objects/square.urdf (robot description, URDF)
Before this commit: robot cube.urdf, 1 links, 0 joints
Links:
- link baseLink: geometry collision mesh filename=square.obj scale=1 1 1; visual mesh filename=square.obj scale=1 1 1

File: assets/objects/triangle_small.urdf (robot description, URDF)
Before this commit: robot cube.urdf, 1 links, 0 joints
Links:
- link baseLink: mass 0.2 -> 0.5; geometry collision mesh filename=triangle.STL scale=0.001 0.01 0.001; visual mesh filename=triangle.STL scale=0.001 0.01 0.001
