Commit message: update save contact_px + depth

File: assets/objects/ellipse1.urdf (robot description, URDF)
Before this commit: robot ellipsoid.urdf, 1 links, 0 joints
Links:
- removed link ellipsoid
- added link base_link, mass .1; collision mesh filename=ellipse.obj scale=1 1 1; visual mesh filename=ellipse.obj scale=1 1 1

File: assets/objects/hexagon.urdf (robot description, URDF)
Before this commit: robot cube.urdf, 1 links, 0 joints
Links:
- removed link baseLink
- added link hexagonal_prism, mass .1; collision mesh filename=hexagonal_prism_rounded.obj scale=0.03 0.03 0.03; visual mesh filename=hexagonal_prism_rounded.obj scale=0.03 0.03 0.03

File: assets/objects/hexagon1.urdf (robot description, URDF)
Before this commit: robot cube.urdf, 1 links, 0 joints
Links:
- link baseLink: geometry collision mesh filename=hexagon.obj scale=1 1 1; visual mesh filename=hexagon.obj scale=1 1 1

File: assets/objects/sphere3.urdf (robot description, URDF)
Before this commit: robot urdf_robot, 1 links, 0 joints
Links:
- link base_link: geometry collision sphere radius=0.003; visual mesh filename=textured_sphere_smooth.obj scale=0.003 0.003 0.003
