Commit message: after calib

File: assets/objects/cube_small.urdf (robot description, URDF)
Before this commit: robot cube.urdf, 1 links, 0 joints
Links:
- link baseLink: geometry collision box size=.05 .05 .05; visual mesh filename=cube.obj scale=.05 .05 .05

Commit message: up2date

File: assets/objects/cube_small.urdf (robot description, URDF)
Before this commit: robot cube.urdf, 1 links, 0 joints
Links:
- link baseLink: geometry collision box size=.025 .025 .025; visual mesh filename=cube.obj scale=.025 .025 .025

File: assets/objects/sphere_25.urdf (robot description, URDF)
Before this commit: robot urdf_robot, 1 links, 0 joints
Links:
- link base_link: geometry collision sphere radius=0.025; visual mesh filename=textured_sphere_smooth.obj scale=0.025 0.025 0.025

Commit message: test

File: assets/objects/cube_small.urdf (robot description, URDF)
Before this commit: robot cube.urdf, 1 links, 0 joints
Links:
- link baseLink: geometry collision box size=.0025 .0025 .0025; visual mesh filename=cube.obj scale=.0025 .0025 .0025

File: assets/objects/ellipse_small.urdf (robot description, URDF)
Before this commit: robot urdf_robot, 1 links, 0 joints
Links:
- link base_link: geometry collision sphere radius=0.002; visual mesh filename=textured_sphere_smooth.obj scale=0.002 0.002 0.0002

Commit message: fixed logging

File: assets/objects/cube_small.urdf (robot description, URDF)
Before this commit: robot cube.urdf, 1 links, 0 joints
Links:
- link baseLink: geometry collision box size=.004 .004 .004; visual mesh filename=cube.obj scale=.004 .004 .004

File: assets/objects/ellipse_small.urdf (robot description, URDF)
Before this commit: robot urdf_robot, 1 links, 0 joints
Links:
- link base_link: geometry collision sphere radius=0.004; visual mesh filename=textured_sphere_smooth.obj scale=0.004 0.004 0.002

File: assets/objects/rect_small.urdf (robot description, URDF)
Before this commit: robot cube.urdf, 1 links, 0 joints
Links:
- link baseLink: geometry collision box size=.004 .004 .001; visual mesh filename=cube.obj scale=.004 .004 .001

Commit message: added some games

File: assets/objects/cube_small.urdf (robot description, URDF)
Before this commit: robot cube.urdf, 1 links, 0 joints
Links:
- link baseLink: geometry collision box size=.004 .004 .004; visual mesh filename=cube.obj scale=.004 .004 .004

File: assets/objects/ellipse_small.urdf (robot description, URDF)
Before this commit: robot urdf_robot, 1 links, 0 joints
Links:
- link base_link: geometry collision sphere radius=0.004; visual mesh filename=textured_sphere_smooth.obj scale=0.004 0.004 0.002

File: assets/objects/rect_small.urdf (robot description, URDF)
Before this commit: robot cube.urdf, 1 links, 0 joints
Links:
- link baseLink: geometry collision box size=.004 .004 .002; visual mesh filename=cube.obj scale=.004 .004 .002

Commit message: fixed constraint type

File: assets/objects/cube_small.urdf (robot description, URDF)
Before this commit: robot cube.urdf, 1 links, 0 joints
Links:
- link baseLink: geometry collision box size=0.004 0.004 0.004; visual mesh filename=cube.obj scale=0.004 0.004 0.004

Commit message: added depth press option

File: assets/objects/cube_small.urdf (robot description, URDF)
Before this commit: robot cube.urdf, 1 links, 0 joints
Links:
- link baseLink: mass 1 -> 0.5

File: assets/objects/ellipse_small.urdf (robot description, URDF)
Before this commit: robot urdf_robot, 1 links, 0 joints
Links:
- link base_link: geometry collision sphere radius=0.004; visual mesh filename=textured_sphere_smooth.obj scale=0.004 0.004 0.002

Commit message: sim update

File: assets/objects/cube_small.urdf (robot description, URDF)
Before this commit: robot cube.urdf, 1 links, 0 joints
Links:
- link baseLink: mass 0.5 -> 0.2; geometry collision box size=0.004 0.004 0.002; visual mesh filename=cube.obj scale=0.004 0.004 0.002

File: assets/objects/rect_small.urdf (robot description, URDF)
Before this commit: robot cube.urdf, 1 links, 0 joints
Links:
- link baseLink: mass 1 -> 0.2; geometry collision box size=.004 .004 .002; visual mesh filename=cube.obj scale=.004 .004 .002

Commit message: fixed collision problems

File: assets/objects/cube_small.urdf (robot description, URDF)
Before this commit: robot cube.urdf, 1 links, 0 joints
Links:
- link baseLink: mass 0.2 -> 0.1
