Commit message: tests

File: assets/objects/rect_grasp.urdf (robot description, URDF)
Before this commit: robot cube.urdf, 1 links, 0 joints
Links:
- link baseLink: mass 0.01 -> 0.02

File: assets/robots/iiwa14_openhand.urdf (robot description, URDF)
Before this commit: robot iiwa14, 21 links, 20 joints
Links:
- removed link iiwa_hand_cam_origin
- removed link iiwa_mocap_link_1
- removed link iiwa_mocap_link_2
Joints:
- removed joint iiwa_gripper_mocap_joint1
- removed joint iiwa_gripper_mocap_joint2
- removed joint iiwa_hand_cam_joint
- joint base_to_finger_1_1: limit lower=0 upper=1.57079632679 effort=10 velocity=10 -> lower=0 upper=1.57079632679 effort=100 velocity=2
- joint base_to_finger_2_1: limit lower=-1.57079632679 upper=0 effort=10 velocity=10 -> lower=-1.57079632679 upper=0 effort=100 velocity=2
- joint base_to_finger_3_2: limit lower=-0.1 upper=3.0 effort=10 velocity=10 -> lower=-0.1 upper=3.0 effort=100 velocity=2
- joint finger_1_1_to_finger_1_2: limit lower=-0.1 upper=3.0 effort=10.0 velocity=10 -> lower=-0.1 upper=3.0 effort=100 velocity=2; origin xyz=-0.02 +0.00725 0 rpy=0 0 0 -> xyz=-0.02 0.00725 0 rpy=0 0 0
- joint finger_1_2_to_finger_1_3: axis 0 0 1 -> 0 1 0; limit lower=0.0 upper=1.27 effort=10.0 velocity=10 -> lower=0.0 upper=0.5 effort=100 velocity=2; origin xyz=0.000800 0.062 0 rpy=0 0 1.57079632679 -> xyz=0.000800 0.072 0 rpy=1.57079632679 0 1.57079632679
- joint finger_2_1_to_finger_2_2: limit lower=-0.1 upper=3.0 effort=10 velocity=10 -> lower=-0.1 upper=3.0 effort=100 velocity=2; origin xyz=-0.02 +0.00725 0 rpy=0 0 0 -> xyz=-0.02 0.00725 0 rpy=0 0 0
- joint finger_2_2_to_finger_2_3: axis 0 0 1 -> 0 1 0; limit lower=0.0 upper=1.27 effort=10 velocity=10 -> lower=0.0 upper=0.5 effort=100 velocity=2; origin xyz=0.000800 0.062 0 rpy=0 0 1.57079632679 -> xyz=0.000800 0.072 0 rpy=1.57079632679 0 1.57079632679
- joint finger_3_2_to_finger_3_3: axis 0 0 1 -> 0 1 0; limit lower=0.0 upper=1.27 effort=10 velocity=10 -> lower=0.0 upper=0.5 effort=100 velocity=2; origin xyz=0.000800 0.062 0 rpy=0 0 1.57079632679 -> xyz=0.000800 0.072 0 rpy=1.57079632679 0 1.57079632679
