Commit message: games

File: assets/robots/yale_openhand_O/urdf/model.urdf (robot description, URDF)
Before this commit: robot openhand, 11 links, 10 joints
Links:
- removed link camera
- removed link tool_frame
- link finger_1_3: mass None -> 0.1
- link finger_2_3: mass None -> 0.1
- link finger_3_3: mass None -> 0.1
Joints:
- removed joint camera_joint
- removed joint tool_frame_joint
